File: pcb/daughterboard/drivers2.kicad_sch (KiCad schematic)
At the start: 12 parts, among them IC5 TLE94112ESXUMA1, IC6 TLE94112ESXUMA1, IC7 TLE94112ESXUMA1

Commit message: changing powerline
Connections:
- net +9V renamed +5.5V
Changed lines of the file:
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@@
 		)
 	)
-	(label "+9V"
+	(label "+5.5V"
 		(at 102.87 69.85 180)
 		(effects
@@
 		)
 	)
-	(label "+9V"
+	(label "+5.5V"
 		(at 36.83 110.49 180)
 		(effects
@@
 		)
 	)
-	(label "+9V"
+	(label "+5.5V"
 		(at 182.88 69.85 180)
 		(effects
@@
 		)
 	)
-	(label "+9V"
+	(label "+5.5V"
 		(at 262.89 57.15 180)
 		(effects
@@
 		)
 	)
-	(label "+9V"
+	(label "+5.5V"
 		(at 245.11 99.06 180)
 		(effects
@@
 		)
 	)
-	(label "+9V"
+	(label "+5.5V"
 		(at 182.88 57.15 180)
 		(effects
@@
 		)
 	)
-	(label "+9V"
+	(label "+5.5V"
 		(at 102.87 57.15 180)
 		(effects
@@
 		)
 	)
-	(label "+9V"
+	(label "+5.5V"
 		(at 168.91 99.06 180)
 		(effects
@@
 		)
 	)
-	(label "+9V"
+	(label "+5.5V"
 		(at 85.09 99.06 180)
 		(effects
@@
 		)
 	)
-	(label "+9V"
+	(label "+5.5V"
 		(at 262.89 69.85 180)
 		(effects
@@
 			)
 		)
-		(property "Value" "+9V"
+		(property "Value" "+5.5V"
 			(at 21.59 110.4899 90)
 			(show_name no)

Commit message: addec electrolytic capacitors on 5v5 line
Parts:
- added C24: 220uF, A_HANU_FOOTPRINTS:EEE1AA101SP, symbol EEE0JA221WP:EEE0JA221WP
Connections:
- net +5.5V: now also C24.1 (+)
- net GND: now also C24.2 (-)

Commit message: added initial power lines
Parts:
- removed C24: 220uF, A_HANU_FOOTPRINTS:EEE1AA101SP, symbol EEE0JA221WP:EEE0JA221WP

Commit message: Initial pcb design for daughterboard Added 3D models for components Modified the daughterboard to motherboard connectors Removed 220uF capacitors from the 5V5 power line
Parts:
- C13, C14, C16, C17, C19, C20: footprint A_HANU_FOOTPRINTS:CAPC0402X22N -> C0603C104K3RACAUTO:C0603
- C15, C18, C21: footprint A_HANU_FOOTPRINTS:T491A -> LIB_T491A106K016AT:T491A
Changed lines of the file:
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@@
 	(wire
 		(pts
-			(xy 90.17 57.15) (xy 102.87 57.15)
+			(xy 25.4 116.84) (xy 39.37 116.84)
 		)
 		(stroke
@@
 	(wire
 		(pts
-			(xy 90.17 77.47) (xy 102.87 77.47)
+			(xy 90.17 57.15) (xy 102.87 57.15)
 		)
 		(stroke
@@
 	(wire
 		(pts
-			(xy 250.19 59.69) (xy 257.81 59.69)
+			(xy 90.17 77.47) (xy 102.87 77.47)
 		)
 		(stroke
@@
 	(wire
 		(pts
-			(xy 147.32 99.06) (xy 147.32 102.87)
+			(xy 250.19 59.69) (xy 257.81 59.69)
 		)
 		(stroke
@@
 	(wire
 		(pts
-			(xy 72.39 91.44) (xy 78.74 91.44)
+			(xy 147.32 99.06) (xy 147.32 102.87)
 		)
 		(stroke
@@
 	(wire
 		(pts
-			(xy 223.52 107.95) (xy 223.52 110.49)
+			(xy 72.39 91.44) (xy 78.74 91.44)
 		)
 		(stroke
@@
 	(wire
 		(pts
-			(xy 242.57 109.22) (xy 242.57 113.03)
+			(xy 223.52 107.95) (xy 223.52 110.49)
 		)
 		(stroke
@@
 	(wire
 		(pts
-			(xy 25.4 110.49) (xy 36.83 110.49)
+			(xy 242.57 109.22) (xy 242.57 113.03)
 		)
 		(stroke
@@
 	(wire
 		(pts
-			(xy 87.63 104.14) (xy 87.63 101.6)
+			(xy 25.4 119.38) (xy 39.37 119.38)
 		)
 		(stroke
@@
 	(wire
 		(pts
-			(xy 25.4 106.68) (xy 36.83 106.68)
+			(xy 87.63 104.14) (xy 87.63 101.6)
 		)
 		(stroke
@@
 	)
 	(label "+3.3V"
-		(at 36.83 106.68 180)
+		(at 39.37 116.84 180)
 		(effects
 			(font
@@
 	)
 	(label "+5.5V"
-		(at 36.83 110.49 180)
+		(at 39.37 119.38 180)
 		(effects
 			(font
@@
 			)
 		)
-		(property "Footprint" "A_HANU_FOOTPRINTS:T491A"
+		(property "Footprint" "LIB_T491A106K016AT:T491A"
 			(at 247.65 106.68 0)
 			(hide yes)
@@
 			)
 		)
-		(property "Footprint" "A_HANU_FOOTPRINTS:T491A"
+		(property "Footprint" "LIB_T491A106K016AT:T491A"
 			(at 171.45 106.68 0)
 			(hide yes)
@@
 	(symbol
 		(lib_id "power:+3.3V")
-		(at 25.4 106.68 90)
+		(at 25.4 116.84 90)
 		(unit 1)
 		(body_style 1)
@@
 		(fields_autoplaced yes)
 		(property "Reference" "#PWR028"
-			(at 29.21 106.68 0)
+			(at 29.21 116.84 0)
 			(hide yes)
 			(show_name no)
@@
 		)
 		(property "Value" "+3.3V"
-			(at 21.59 106.6799 90)
+			(at 21.59 116.8399 90)
 			(show_name no)
 			(do_not_autoplace no)
@@
 		)
 		(property "Footprint" ""
-			(at 25.4 106.68 0)
+			(at 25.4 116.84 0)
 			(hide yes)
 			(show_name no)
@@
 		)
 		(property "Datasheet" ""
-			(at 25.4 106.68 0)
+			(at 25.4 116.84 0)
 			(hide yes)
 			(show_name no)
@@
 		)
 		(property "Description" "Power symbol creates a global label with name \"+3.3V\""
-			(at 25.4 106.68 0)
+			(at 25.4 116.84 0)
 			(hide yes)
 			(show_name no)
@@
 			)
 		)
-		(property "Footprint" "A_HANU_FOOTPRINTS:CAPC0402X22N"
+		(property "Footprint" "C0603C104K3RACAUTO:C0603"
 			(at 242.57 106.68 0)
 			(hide yes)
@@
 			)
 		)
-		(property "Footprint" "A_HANU_FOOTPRINTS:CAPC0402X22N"
+		(property "Footprint" "C0603C104K3RACAUTO:C0603"
 			(at 63.5 105.41 0)
 			(hide yes)
@@
 			)
 		)
-		(property "Footprint" "A_HANU_FOOTPRINTS:T491A"
+		(property "Footprint" "LIB_T491A106K016AT:T491A"
 			(at 87.63 106.68 0)
 			(hide yes)
@@
 			)
 		)
-		(property "Footprint" "A_HANU_FOOTPRINTS:CAPC0402X22N"
+		(property "Footprint" "C0603C104K3RACAUTO:C0603"
 			(at 166.37 106.68 0)
 			(hide yes)
@@
 			)
 		)
-		(property "Footprint" "A_HANU_FOOTPRINTS:CAPC0402X22N"
+		(property "Footprint" "C0603C104K3RACAUTO:C0603"
 			(at 223.52 105.41 0)
 			(hide yes)
@@
 	(symbol
 		(lib_id "power:+9V")
-		(at 25.4 110.49 90)
+		(at 25.4 119.38 90)
 		(unit 1)
 		(body_style 1)
@@
 		(fields_autoplaced yes)
 		(property "Reference" "#PWR029"
-			(at 29.21 110.49 0)
+			(at 29.21 119.38 0)
 			(hide yes)
 			(show_name no)
@@
 		)
 		(property "Value" "+5.5V"
-			(at 21.59 110.4899 90)
+			(at 21.59 119.3799 90)
 			(show_name no)
 			(do_not_autoplace no)
@@
 		)
 		(property "Footprint" ""
-			(at 25.4 110.49 0)
+			(at 25.4 119.38 0)
 			(hide yes)
 			(show_name no)
@@
 		)
 		(property "Datasheet" ""
-			(at 25.4 110.49 0)
+			(at 25.4 119.38 0)
 			(hide yes)
 			(show_name no)
@@
 		)
 		(property "Description" "Power symbol creates a global label with name \"+9V\""
-			(at 25.4 110.49 0)
+			(at 25.4 119.38 0)
 			(hide yes)
 			(show_name no)
@@
 			)
 		)
-		(property "Footprint" "A_HANU_FOOTPRINTS:CAPC0402X22N"
+		(property "Footprint" "C0603C104K3RACAUTO:C0603"
 			(at 82.55 106.68 0)
 			(hide yes)
@@
 			)
 		)
-		(property "Footprint" "A_HANU_FOOTPRINTS:CAPC0402X22N"
+		(property "Footprint" "C0603C104K3RACAUTO:C0603"
 			(at 147.32 105.41 0)
 			(hide yes)

Commit message: Finalized daughterboard pcb design 0 errors Verified every 3D model, footprint According to the schematic
Parts:
- IC5, IC6, IC7: footprint A_HANU_FOOTPRINTS:TLE94112ESXUMA1 -> driver_tle:SOP65P600X115-25N
Changed lines of the file:
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@@
 	)
 	(hierarchical_label "SPI_MISO"
-		(shape input)
+		(shape output)
 		(at 54.61 64.77 180)
 		(effects
@@
 			)
 		)
-		(property "Footprint" "A_HANU_FOOTPRINTS:TLE94112ESXUMA1"
+		(property "Footprint" "driver_tle:SOP65P600X115-25N"
 			(at 166.37 144.45 0)
 			(hide yes)
@@
 			)
 		)
-		(property "Footprint" "A_HANU_FOOTPRINTS:TLE94112ESXUMA1"
+		(property "Footprint" "driver_tle:SOP65P600X115-25N"
 			(at 246.38 144.45 0)
 			(hide yes)
@@
 			)
 		)
-		(property "Footprint" "A_HANU_FOOTPRINTS:TLE94112ESXUMA1"
+		(property "Footprint" "driver_tle:SOP65P600X115-25N"
 			(at 86.36 144.45 0)
 			(hide yes)

Commit message: Final touches for the PCB order Added MPN, Description, checked footprints and 3D models Finished the BOM
Parts:
- C13, C14, C16, C17, C19, C20: Manufacturer_Name (none) -> KEMET; Manufacturer_Part_Number (none) -> C0603C104K3RACAUTO
- C15, C18, C21: Manufacturer_Name (none) -> KEMET; Manufacturer_Part_Number (none) -> T491A106K016AT
Changed lines of the file:
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@@
+			)
+		)
+		(property "Manufacturer_Name" "KEMET"
+			(at 247.65 106.68 0)
+			(hide yes)
+			(show_name no)
+			(do_not_autoplace no)
+			(effects
+				(font
+					(size 1.27 1.27)
+				)
+			)
+		)
+		(property "Manufacturer_Part_Number" "T491A106K016AT"
+			(at 247.65 106.68 0)
+			(hide yes)
+			(show_name no)
+			(do_not_autoplace no)
+			(effects
+				(font
+					(size 1.27 1.27)
+				)
 			)
 		)
@@
 			)
 		)
+		(property "Manufacturer_Name" "KEMET"
+			(at 171.45 106.68 0)
+			(hide yes)
+			(show_name no)
+			(do_not_autoplace no)
+			(effects
+				(font
+					(size 1.27 1.27)
+				)
+			)
+		)
+		(property "Manufacturer_Part_Number" "T491A106K016AT"
+			(at 171.45 106.68 0)
+			(hide yes)
+			(show_name no)
+			(do_not_autoplace no)
+			(effects
+				(font
+					(size 1.27 1.27)
+				)
+			)
+		)
 		(pin "1"
 		)
@@
 			)
 		)
+		(property "Manufacturer_Name" "KEMET"
+			(at 242.57 106.68 0)
+			(hide yes)
+			(show_name no)
+			(do_not_autoplace no)
+			(effects
+				(font
+					(size 1.27 1.27)
+				)
+			)
+		)
+		(property "Manufacturer_Part_Number" "C0603C104K3RACAUTO"
+			(at 242.57 106.68 0)
+			(hide yes)
+			(show_name no)
+			(do_not_autoplace no)
+			(effects
+				(font
+					(size 1.27 1.27)
+				)
+			)
+		)
 		(pin "1"
 		)
@@
 			)
 		)
+		(property "Manufacturer_Name" "KEMET"
+			(at 63.5 105.41 0)
+			(hide yes)
+			(show_name no)
+			(do_not_autoplace no)
+			(effects
+				(font
+					(size 1.27 1.27)
+				)
+			)
+		)
+		(property "Manufacturer_Part_Number" "C0603C104K3RACAUTO"
+			(at 63.5 105.41 0)
+			(hide yes)
+			(show_name no)
+			(do_not_autoplace no)
+			(effects
+				(font
+					(size 1.27 1.27)
+				)
+			)
+		)
 		(pin "2"
 		)
@@
 			)
 		)
+		(property "Manufacturer_Name" "KEMET"
+			(at 87.63 106.68 0)
+			(hide yes)
+			(show_name no)
+			(do_not_autoplace no)
+			(effects
+				(font
+					(size 1.27 1.27)
+				)
+			)
+		)
+		(property "Manufacturer_Part_Number" "T491A106K016AT"
+			(at 87.63 106.68 0)
+			(hide yes)
+			(show_name no)
+			(do_not_autoplace no)
+			(effects
+				(font
+					(size 1.27 1.27)
+				)
+			)
+		)
 		(pin "1"
 		)
@@
 			)
 		)
+		(property "Manufacturer_Name" "KEMET"
+			(at 166.37 106.68 0)
+			(hide yes)
+			(show_name no)
+			(do_not_autoplace no)
+			(effects
+				(font
+					(size 1.27 1.27)
+				)
+			)
+		)
+		(property "Manufacturer_Part_Number" "C0603C104K3RACAUTO"
+			(at 166.37 106.68 0)
+			(hide yes)
+			(show_name no)
+			(do_not_autoplace no)
+			(effects
+				(font
+					(size 1.27 1.27)
+				)
+			)
+		)
 		(pin "1"
 		)
@@
 			)
 		)
+		(property "Manufacturer_Name" "KEMET"
+			(at 223.52 105.41 0)
+			(hide yes)
+			(show_name no)
+			(do_not_autoplace no)
+			(effects
+				(font
+					(size 1.27 1.27)
+				)
+			)
+		)
+		(property "Manufacturer_Part_Number" "C0603C104K3RACAUTO"
+			(at 223.52 105.41 0)
+			(hide yes)
+			(show_name no)
+			(do_not_autoplace no)
+			(effects
+				(font
+					(size 1.27 1.27)
+				)
+			)
+		)
 		(pin "2"
 		)
@@
 			)
 		)
+		(property "Manufacturer_Name" "KEMET"
+			(at 82.55 106.68 0)
+			(hide yes)
+			(show_name no)
+			(do_not_autoplace no)
+			(effects
+				(font
+					(size 1.27 1.27)
+				)
+			)
+		)
+		(property "Manufacturer_Part_Number" "C0603C104K3RACAUTO"
+			(at 82.55 106.68 0)
+			(hide yes)
+			(show_name no)
+			(do_not_autoplace no)
+			(effects
+				(font
+					(size 1.27 1.27)
+				)
+			)
+		)
 		(pin "1"
 		)
@@
 			(at 147.32 105.41 0)
 			(hide yes)
+			(show_name no)
+			(do_not_autoplace no)
+			(effects
+				(font
+					(size 1.27 1.27)
+				)
+			)
+		)
+		(property "Manufacturer_Name" "KEMET"
+			(at 147.32 105.41 0)
+			(hide yes)
+			(show_name no)
+			(do_not_autoplace no)
+			(effects
+				(font
+					(size 1.27 1.27)
+				)
+			)
+		)
+		(property "Manufacturer_Part_Number" "C0603C104K3RACAUTO"
+			(at 147.32 105.41 0)
+			(hide yes)
