File: pcb/daughterboard/daughterboard.kicad_sch (KiCad schematic)
At the start: 2 parts, among them J2 M20-7820646, J23 Screw_Terminal_01x03

Commit message: updated MPN in BOM
Parts:
- J23: Manufacturer_Part_Number M20-7820646 -> 1729131
Changed lines of the file:
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@@
 			)
 		)
-		(property "Manufacturer_Part_Number" "M20-7820646"
+		(property "Manufacturer_Part_Number" "1729131"
 			(at 163.83 68.58 0)
 			(hide yes)

Commit message: modified motor connectors
Parts:
- renumbered J23 to J1
Changed lines of the file:
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@@
 		(in_pos_files yes)
 		(dnp no)
-		(property "Reference" "J23"
+		(property "Reference" "J1"
 			(at 162.814 59.944 0)
 			(show_name no)
@@
 			(project "daughterboard"
 				(path "/2255186e-2dec-4723-baeb-acb5f2843560"
-					(reference "J23")
+					(reference "J1")
 					(unit 1)
 				)
