File: pcb/motherboard/motherboard.kicad_pcb (KiCad board)
At the start: 2 copper layers, 100 x 100 mm, 95 parts, among them J1 BOOT PIN HEADER, J10 Conn_01x04, J11 M20-7820646, J13 M20-7820646, J15 M20-7820646, J17 Terminal 1, J18 Terminal 2, J19 Terminal Block, J2 ST-Link, J20 Terminal Block, J21 Terminal Block, J22 Terminal Block, J23 Terminal Block, J3 UART_USB, J4 I2C_HEADER, J5 KPJX-4S-S, J6 SPI_TEST, J7 M20-7820646, J8 Conn_01x04, J9 M20-7820646, SW1 STM_RST, SW2 GEN_MAZE, SW3 TOGGLE_MAZE, SW4 SOLVE_MAZE, U1 STM32F103C8Tx, U2 CH340C, U3 TPS5420D, U4 TPS5420D, U5 AMS1117-3.3, U6 PCA9306D, U7 74HC138, Y1 8MHz, Y2 32.768KHz

Commit message: motherboard PCB fixes
Routing:
- net /SOLVE_MAZE: track 23.3 -> 19.7 mm
Changed lines of the file:
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@@
 		)
 		(embedded_fonts no)
-		(model "${KICAD10_3DMODEL_DIR}/Connector_USB.3dshapes/USB_C_Receptacle_HRO_TYPE-C-31-M-12.step"
+		(model "/home/joey/work/dev/tilting-maze/pcb/lib/usbc_3d_model/HRO_TYPE-C-31-M-12.step"
 			(offset
-				(xyz 0 0 0)
+				(xyz -4.445 -3.175 0)
 			)
 			(scale
@@
 			)
 			(rotate
-				(xyz 0 0 0)
+				(xyz -0 -0 -0)
 			)
 		)
@@
 		(net "/SOLVE_MAZE")
 	)
-	(segment
-		(start 137.16 67.564)
-		(end 140.716 67.564)
-		(width 0.2)
-		(layer "B.Cu")
-		(net "/SOLVE_MAZE")
-	)
