File: pcb/motherboard/motherboard.kicad_pcb (KiCad board)
At the start: 2 copper layers, 100 x 100 mm, 95 parts, among them J1 BOOT PIN HEADER, J10 Conn_01x04, J11 M20-7820646, J13 M20-7820646, J15 M20-7820646, J17 Terminal 1, J18 Terminal 2, J19 Terminal Block, J2 ST-Link, J20 Terminal Block, J21 Terminal Block, J22 Terminal Block, J23 Terminal Block, J3 UART_USB, J4 I2C_HEADER, J5 KPJX-4S-S, J6 SPI_TEST, J7 M20-7820646, J8 Conn_01x04, J9 M20-7820646, SW1 STM_RST, SW2 GEN_MAZE, SW3 TOGGLE_MAZE, SW4 SOLVE_MAZE, U1 STM32F103C8Tx, U2 CH340C, U3 TPS5420D, U4 TPS5420D, U5 AMS1117-3.3, U6 PCA9306D, U7 74HC138, Y1 8MHz, Y2 32.768KHz

Commit message: replaced PCA9306D component on motherboard
Parts:
- U6: footprint Package_SO:SO-8_3.9x4.9mm_P1.27mm -> Package_SON:X2SON-8_1.4x1mm_P0.35mm
- moved C26 2.16 mm to (159.1, 77.9)
Routing:
- net Net-(U6-EN): track 6.63 -> 11.9 mm
- net /STM32/PB11: track 16.2 -> 20.5 mm, vias 2 -> 4
- net GND: track 116.7 -> 113.1 mm, vias 297 -> 304
- net Net-(J4-Pin_3): track 6.52 -> 9.33 mm
- net Net-(J4-Pin_2): track 6.71 -> 9.14 mm
- net +3V3: track 526.9 -> 529.3 mm
- net /STM32/PB10: track 17.8 -> 18.8 mm
