File: pcb/motherboard/stm32.kicad_sch (KiCad schematic)
At the start: 18 parts, among them J1 BOOT PIN HEADER, J2 ST-Link, SW1 STM_RST, U1 STM32F103C8Tx, Y1 8MHz, Y2 32.768KHz

Commit message: added almost all footprints for PCB design
Parts:
- C10, C5, C6, C7, C8, C9: footprint (none) -> Capacitor_SMD:C_0603_1608Metric
- J1: footprint (none) -> Connector_PinHeader_2.54mm:PinHeader_1x03_P2.54mm_Vertical
- J2: footprint Connector:FanPinHeader_1x04_P2.54mm_Vertical -> Connector_PinHeader_2.54mm:PinHeader_1x04_P2.54mm_Vertical
- R1, R2: footprint (none) -> Resistor_SMD:R_0603_1608Metric
- SW1: footprint (none) -> Connector_PinHeader_2.54mm:PinHeader_1x02_P2.54mm_Vertical
- Y1, Y2: footprint (none) -> Crystal:Crystal_SMD_3215-2Pin_3.2x1.5mm
Changed lines of the file:
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@@
 			)
 		)
-		(property "Footprint" "Connector:FanPinHeader_1x04_P2.54mm_Vertical"
+		(property "Footprint" "Connector_PinHeader_2.54mm:PinHeader_1x04_P2.54mm_Vertical"
 			(at 181.61 133.35 0)
 			(hide yes)
@@
 			)
 		)
-		(property "Footprint" ""
+		(property "Footprint" "Capacitor_SMD:C_0603_1608Metric"
 			(at 228.6 48.26 0)
 			(hide yes)
@@
 			)
 		)
-		(property "Footprint" ""
+		(property "Footprint" "Connector_PinHeader_2.54mm:PinHeader_1x03_P2.54mm_Vertical"
 			(at 212.09 133.35 0)
 			(hide yes)
@@
 			)
 		)
-		(property "Footprint" ""
+		(property "Footprint" "Capacitor_SMD:C_0603_1608Metric"
 			(at 80.01 129.54 0)
 			(hide yes)
@@
 			)
 		)
-		(property "Footprint" ""
+		(property "Footprint" "Connector_PinHeader_2.54mm:PinHeader_1x02_P2.54mm_Vertical"
 			(at 67.31 129.54 0)
 			(hide yes)
@@
 			)
 		)
-		(property "Footprint" ""
+		(property "Footprint" "Capacitor_SMD:C_0603_1608Metric"
 			(at 195.58 48.26 0)
 			(hide yes)
@@
 			)
 		)
-		(property "Footprint" ""
+		(property "Footprint" "Crystal:Crystal_SMD_3215-2Pin_3.2x1.5mm"
 			(at 55.88 46.99 0)
 			(hide yes)
@@
 			)
 		)
-		(property "Footprint" ""
+		(property "Footprint" "Capacitor_SMD:C_0603_1608Metric"
 			(at 184.15 48.26 0)
 			(hide yes)
@@
 			)
 		)
-		(property "Footprint" ""
+		(property "Footprint" "Capacitor_SMD:C_0603_1608Metric"
 			(at 207.01 48.26 0)
 			(hide yes)
@@
 			)
 		)
-		(property "Footprint" ""
+		(property "Footprint" "Resistor_SMD:R_0603_1608Metric"
 			(at 224.79 133.35 0)
 			(hide yes)
@@
 			)
 		)
-		(property "Footprint" ""
+		(property "Footprint" "Capacitor_SMD:C_0603_1608Metric"
 			(at 217.17 48.26 0)
 			(hide yes)
@@
 			)
 		)
-		(property "Footprint" ""
+		(property "Footprint" "Resistor_SMD:R_0603_1608Metric"
 			(at 67.31 121.92 0)
 			(hide yes)
@@
 			)
 		)
-		(property "Footprint" ""
+		(property "Footprint" "Crystal:Crystal_SMD_3215-2Pin_3.2x1.5mm"
 			(at 55.88 74.93 0)
 			(hide yes)

Commit message: consolidated BOM for motherboard, added terminal blocks for external motors
Parts:
- C1, C2, C3, C4: footprint Capacitor_SMD:C_0201_0603Metric -> Capacitor_SMD:C_0603_1608Metric
Changed lines of the file:
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@@
 			)
 		)
-		(property "Footprint" "Capacitor_SMD:C_0201_0603Metric"
+		(property "Footprint" "Capacitor_SMD:C_0603_1608Metric"
 			(at 49.53 52.07 0)
 			(hide yes)
@@
 			)
 		)
-		(property "Footprint" "Capacitor_SMD:C_0201_0603Metric"
+		(property "Footprint" "Capacitor_SMD:C_0603_1608Metric"
 			(at 62.23 80.01 0)
 			(hide yes)
@@
 			)
 		)
-		(property "Footprint" "Capacitor_SMD:C_0201_0603Metric"
+		(property "Footprint" "Capacitor_SMD:C_0603_1608Metric"
 			(at 49.53 80.01 0)
 			(hide yes)
@@
 			)
 		)
-		(property "Footprint" "Capacitor_SMD:C_0201_0603Metric"
+		(property "Footprint" "Capacitor_SMD:C_0603_1608Metric"
 			(at 62.23 52.07 0)
 			(hide yes)

Commit message: added connectors for external motors, finished most of the motherboard PCB
Parts:
- J2: footprint Connector_PinHeader_2.54mm:PinHeader_1x04_P2.54mm_Vertical -> Connector_PinHeader_2.54mm:PinHeader_1x04_P2.54mm_Horizontal
Connections:
- net SPI_CLK: now also U1.15 (PA5); no longer U1.14 (PA4)
- net SPI_CS: now also U1.14 (PA4); no longer U1.13 (PA3)
- net SPI_MISO: now also U1.16 (PA6); no longer U1.15 (PA5)
- net SPI_MOSI: now also U1.17 (PA7); no longer U1.16 (PA6)
- net PB0: now reaches U1.18 (PB0)
- net PB1: now reaches U1.19 (PB1)
- net PB13: now reaches U1.26 (PB13)
- net PB14: now reaches U1.27 (PB14)
- net PB15: now reaches U1.28 (PB15)
- net PA8: now reaches U1.29 (PA8)
- net PA11: now reaches U1.32 (PA11)
- new net PA3: U1.13 (PA3)
- no-connect marks 14 -> 6
Other:
- note added: "12V Motor 1"
- note added: "12V Motor 2"
- note added: "12V Motor 3"
- note added: "12V Motor 4"
- note added: "PWM"
- moved on the sheet: J1, J2, R1

Commit message: Final touches for the PCB order Added MPN, Description, checked footprints and 3D models Finished the BOM
Parts:
- C1, C2: Manufacturer_Name (none) -> YAGEO; Manufacturer_Part_Number (none) -> CC0603JRNPO9BN200
- C10, C5, C6, C7, C8, C9: Manufacturer_Name (none) -> YAGEO; Manufacturer_Part_Number (none) -> CC0603KRX7R9BB104
- C3, C4: Manufacturer_Name (none) -> YAGEO; Manufacturer_Part_Number (none) -> CC0603JRNPO9BN120
- J1: Manufacturer_Name (none) -> Wurth Elektronik; Manufacturer_Part_Number (none) -> 61300311121
- J2: Manufacturer_Name (none) -> Wurth Elektronik; Manufacturer_Part_Number (none) -> 61300411121
- R1: Manufacturer_Name (none) -> YAGEO; Manufacturer_Part_Number (none) -> RC0603FR-07100KL
- R2: Manufacturer_Name (none) -> YAGEO; Manufacturer_Part_Number (none) -> RC0603FR-0710KL
- SW1: Manufacturer_Name (none) -> Wurth Elektronik; Manufacturer_Part_Number (none) -> 61300211121
- U1: Manufacturer_Name (none) -> STMicroelectronics; Manufacturer_Part_Number (none) -> STM32F103C8T6
- Y1: Manufacturer_Name (none) -> Abracon; Manufacturer_Part_Number (none) -> ABM3C-8.000MHZ-D4Y-T
- Y2: Manufacturer_Name (none) -> Abracon; Manufacturer_Part_Number (none) -> ABS07-120-32.768KHZ-T

Commit message: updated MPN in BOM
Parts:
- C10, C5, C6, C7, C8, C9: Manufacturer_Part_Number CC0603KRX7R9BB104 -> CC0603JRX7R9BB104
- Y1: Manufacturer_Part_Number ABM3C-8.000MHZ-D4Y-T -> FY0800018
Changed lines of the file:
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@@
 			)
 		)
-		(property "Manufacturer_Part_Number" "CC0603KRX7R9BB104"
+		(property "Manufacturer_Part_Number" "CC0603JRX7R9BB104"
 			(at 228.6 48.26 0)
 			(hide yes)
@@
 			)
 		)
-		(property "Manufacturer_Part_Number" "CC0603KRX7R9BB104"
+		(property "Manufacturer_Part_Number" "CC0603JRX7R9BB104"
 			(at 80.01 129.54 0)
 			(hide yes)
@@
 			)
 		)
-		(property "Manufacturer_Part_Number" "CC0603KRX7R9BB104"
+		(property "Manufacturer_Part_Number" "CC0603JRX7R9BB104"
 			(at 195.58 48.26 0)
 			(hide yes)
@@
 			)
 		)
-		(property "Manufacturer_Part_Number" "ABM3C-8.000MHZ-D4Y-T"
+		(property "Manufacturer_Part_Number" "FY0800018"
 			(at 55.88 46.99 0)
 			(hide yes)
@@
 			)
 		)
-		(property "Manufacturer_Part_Number" "CC0603KRX7R9BB104"
+		(property "Manufacturer_Part_Number" "CC0603JRX7R9BB104"
 			(at 184.15 48.26 0)
 			(hide yes)
@@
 			)
 		)
-		(property "Manufacturer_Part_Number" "CC0603KRX7R9BB104"
+		(property "Manufacturer_Part_Number" "CC0603JRX7R9BB104"
 			(at 207.01 48.26 0)
 			(hide yes)
@@
 			)
 		)
-		(property "Manufacturer_Part_Number" "CC0603KRX7R9BB104"
+		(property "Manufacturer_Part_Number" "CC0603JRX7R9BB104"
 			(at 217.17 48.26 0)
 			(hide yes)
